File: schematic/delay_pedal.kicad_sch (KiCad schematic)
At the start: 140 parts, among them J1 IN Gain, J10 VFLASH, J12 LP, J13 Mix, J14 OUT Gain, J3 SPI FLASH, J4 Audio In, J5 FDBK, J6 +9V, J8 Time, J9 Audio Out, SW1 RESET, SW2 SW_SPST, U1 ICE40LP1K-QN84, U10 TPL810ADJ-5TR, U11 TPL810F50-89TR, U12 ADS8339IDGSR, U13 TLV76033DBZR, U14 OPA1678, U15 DAC8551IADGKR, U16 REF5045AD, U17 OPA1678, U2 APS1604M-3SQR, U3 OPA1678, U4 NXB0104, U5 OPA1678, U6 W25X20CLSN, U8 OPA1678, U9 OPA1678, X1 KXO-V96T

Commit message: Added missing capacitors to analog signal chain
Parts:
- added C56: 47u, Capacitor_SMD:C_0603_1608Metric_Pad1.08x0.95mm_HandSolder, symbol Device:C
- added C58, C59: 0.47u, Capacitor_SMD:C_0603_1608Metric_Pad1.08x0.95mm_HandSolder, symbol Device:C
- added C60: 0.1u, Capacitor_SMD:C_0603_1608Metric_Pad1.08x0.95mm_HandSolder, symbol Device:C
- added D3: LED, LED_SMD:LED_0603_1608Metric_Pad1.05x0.95mm_HandSolder, symbol Device:LED
- added R21, R35: 40k, Resistor_SMD:R_0603_1608Metric_Pad0.98x0.95mm_HandSolder, symbol Device:R_US
- added R36: 1M, Resistor_SMD:R_0603_1608Metric_Pad0.98x0.95mm_HandSolder, symbol Device:R_US
- added R37: 1k, Resistor_SMD:R_0603_1608Metric_Pad0.98x0.95mm_HandSolder, symbol Device:R_US
- R12, R13, R14, R31, R32: value 10k -> 20k
- R29, R30: value 10k -> 40k
Connections:
- net +5V: now also R21.1
- net GND: now also C56.2, R35.2, R37.2
- net Vref: now also R36.1; no longer U8.5 (+)
- net at C14.2, R31.2, U8.1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: now also C59.2; no longer R12.1
- net at C15.1, J12.1 (Pin_1): now also C60.1; no longer U9.5 (+)
- net at R23.2, TP5.1, U9.6 (-)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: now also C58.2; no longer J5.1 (Pin_1)
- net ICELED: now reaches U1.A5 (IOL_5B)
- net ICELED: now also D3.2 (A)
- new net: C59.1, R12.1
- new net: C60.2, R36.2, U9.5 (+)
- new net: C58.1, J5.1 (Pin_1)
- new net: D3.1 (K), R37.1
- new net +2V5: C56.1, R21.2, R35.1, U8.5 (+)
- no-connect marks 54 -> 53
Other:
- moved on the sheet: C13, C14, C15, C16, C17, C25, C26, C33, C34, C35, C40, C5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

Commit message: Updated Schottky diode footprint
Parts:
- D6: footprint Diode_SMD:D_0603_1608Metric_Pad1.05x0.95mm_HandSolder -> Diode_SMD:D_SOD-323_HandSoldering
Changed lines of the file:
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@@
 			)
 		)
-		(property "Footprint" "Diode_SMD:D_0603_1608Metric_Pad1.05x0.95mm_HandSolder"
+		(property "Footprint" "Diode_SMD:D_SOD-323_HandSoldering"
 			(at 363.22 262.89 0)
 			(effects

Commit message: Generated fabrication files
Parts:
- C19: footprint Capacitor_SMD:C_0603_1608Metric_Pad1.08x0.95mm_HandSolder -> Capacitor_THT:CP_Radial_D6.3mm_P2.50mm
- C40, C5, C60: footprint Capacitor_SMD:C_0603_1608Metric_Pad1.08x0.95mm_HandSolder -> Capacitor_SMD:C_1206_3216Metric_Pad1.33x1.80mm_HandSolder
- J1, J12, J14, J4, J5, J6, J9: footprint TerminalBlock_Phoenix:TerminalBlock_Phoenix_MPT-0,5-2-2.54_1x02_P2.54mm_Horizontal -> Connector_PinHeader_2.54mm:PinHeader_1x02_P2.54mm_Vertical; symbol Connector:Screw_Terminal_01x02 -> Connector_Generic:Conn_01x02
- J13: footprint TerminalBlock_Phoenix:TerminalBlock_Phoenix_MPT-0,5-3-2.54_1x03_P2.54mm_Horizontal -> Connector_PinHeader_2.54mm:PinHeader_1x03_P2.54mm_Vertical; symbol Connector:Screw_Terminal_01x03 -> Connector_Generic:Conn_01x03
- J8: footprint TerminalBlock_Phoenix:TerminalBlock_Phoenix_MPT-0,5-5-2.54_1x05_P2.54mm_Horizontal -> Connector_PinHeader_2.54mm:PinHeader_1x05_P2.54mm_Vertical; symbol Connector:Screw_Terminal_01x05 -> Connector_Generic:Conn_01x05
- SW2: footprint TerminalBlock_Phoenix:TerminalBlock_Phoenix_MPT-0,5-2-2.54_1x02_P2.54mm_Horizontal -> Connector_PinHeader_2.54mm:PinHeader_1x02_P2.54mm_Vertical
- U14, U17, U3, U5, U8, U9: value OPA1678 -> RC4580; symbol Amplifier_Operational:OPA1678 -> Amplifier_Operational:RC4580

Commit message: Fixed footprint assignments
Parts:
- C35, C56, C58, C59: footprint Capacitor_SMD:C_0603_1608Metric_Pad1.08x0.95mm_HandSolder -> Capacitor_SMD:C_1206_3216Metric_Pad1.33x1.80mm_HandSolder
- U13: footprint PCM_Package_TO_SOT_SMD_AKL:SOT-89-3_Handsoldering -> Package_TO_SOT_SMD:SOT-23-3
Changed lines of the file:
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@@
 			)
 		)
-		(property "Footprint" "Capacitor_SMD:C_0603_1608Metric_Pad1.08x0.95mm_HandSolder"
+		(property "Footprint" "Capacitor_SMD:C_1206_3216Metric_Pad1.33x1.80mm_HandSolder"
 			(at 494.9952 318.77 0)
 			(effects
@@
 			)
 		)
-		(property "Footprint" "Capacitor_SMD:C_0603_1608Metric_Pad1.08x0.95mm_HandSolder"
+		(property "Footprint" "Capacitor_SMD:C_1206_3216Metric_Pad1.33x1.80mm_HandSolder"
 			(at 528.0152 318.77 0)
 			(effects
@@
 			)
 		)
-		(property "Footprint" "PCM_Package_TO_SOT_SMD_AKL:SOT-89-3_Handsoldering"
+		(property "Footprint" "Package_TO_SOT_SMD:SOT-23-3"
 			(at 370.84 389.89 0)
 			(effects
@@
 			)
 		)
-		(property "Footprint" "Capacitor_SMD:C_0603_1608Metric_Pad1.08x0.95mm_HandSolder"
+		(property "Footprint" "Capacitor_SMD:C_1206_3216Metric_Pad1.33x1.80mm_HandSolder"
 			(at 255.5748 64.77 0)
 			(effects
@@
 			)
 		)
-		(property "Footprint" "Capacitor_SMD:C_0603_1608Metric_Pad1.08x0.95mm_HandSolder"
+		(property "Footprint" "Capacitor_SMD:C_1206_3216Metric_Pad1.33x1.80mm_HandSolder"
 			(at 285.75 86.6648 0)
 			(effects
